File: pcb/hackpad.kicad_pcb (KiCad board)
At the start: 2 copper layers, 98 x 124.5 mm, 25 parts, among them J1 Conn_01x04_Pin, SW1 SW_Push, SW11 RotaryEncoder_Switch, SW2 SW_Push, SW3 SW_Push, SW4 SW_Push, SW5 SW_Push, SW6 SW_Push, SW7 SW_Push, SW8 SW_Push, SW9 SW_Push, U1 XIAO-RP2040-SMD

Commit message: Add files via upload
Parts:
- U1: moved to F.Cu
- moved U1 28.4 mm to (151.7, 135.2), turned to 180 degrees
Routing:
- net colunn 0: track 78.7 -> 165.1 mm, vias 0 -> 2
- net S1: track 69.8 -> 143.8 mm, vias 1 -> 5
- net colunn 1: track 58.8 -> 122.4 mm, vias 0 -> 2
- net colunn 2: track 81.5 -> 126.7 mm, vias 0 -> 2
- net A1: track 100.2 -> 144.5 mm, vias 1 -> 2
- net VCC: track 78.2 -> 113.9 mm, vias 1 -> 0
- net SDA: track 151.3 -> 117.0 mm, vias 1 -> 2
- net row 1: track 100.3 -> 123.6 mm, vias 1 -> 2
- net GND: track 111.1 -> 132.5 mm, vias 1 -> 0
- net row 0: track 115.3 -> 131.8 mm, vias 1 -> 4
- net B1: track 84.1 -> 100.4 mm, vias 1 -> 0
- net SCL: track 115.0 -> 118.8 mm, vias 1 -> 0
- net row 2: track 81.9 -> 79.8 mm, vias 1 -> 2
- net Net-(D2-A): track 13.6 -> 15.2 mm, vias 0 -> 2
